File: v0.1/kicad/cheapis.kicad_pcb (KiCad board)
At the start: 2 copper layers, 99.9 x 99.9 mm, 25 parts, among them J1 Conn_01x01, SW1 SW_Diode_Combined, SW10 SW_Diode_Combined, SW11 SW_Diode_Combined, SW12 SW_Diode_Combined, SW13 SW_Diode_Combined, SW14 SW_Diode_Combined, SW15 SW_Diode_Combined, SW16 SW_Diode_Combined, SW17 SW_Diode_Combined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

Commit message: multi-switches-support
Parts:
- SW1, SW10, SW11, SW12, SW13, SW14, SW15, SW16, SW17, SW2, SW3, SW4, SW5, SW6, SW7, SW8, SW9: footprint Redragon:SW_Redragon_LowProfile_PCB_1.00u -> Redragon:MultiSwitches_MX_Redragon_ChocV1
Routing:
- net col4: track 143.9 -> 129.9 mm
- net col5: track 129.0 -> 117.1 mm
- net col3: track 120.4 -> 111.6 mm
- net col2: track 151.9 -> 143.2 mm
- net col1: track 175.1 -> 166.6 mm
Other:
- board text added: "MX_Redragon_Choc"
- board text removed: "But with Redragon Switches"
