File: v0.1/kicad/cheapis.kicad_pcb (KiCad board)
At the start: 2 copper layers, 99.9 x 99.9 mm, 25 parts, among them J1 Conn_01x01, SW1 SW_Diode_Combined, SW10 SW_Diode_Combined, SW11 SW_Diode_Combined, SW12 SW_Diode_Combined, SW13 SW_Diode_Combined, SW14 SW_Diode_Combined, SW15 SW_Diode_Combined, SW16 SW_Diode_Combined, SW17 SW_Diode_Combined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

Commit message: fix some major design problem, rows not fully connected
Routing:
- net col3: track 120.4 -> 123.3 mm
- net col5: track 129.0 -> 131.8 mm
- net col2: track 151.9 -> 153.5 mm
- net col1: track 175.1 -> 176.8 mm
